File: KiCad/Project/EEG_BLE.sch (KiCad schematic (older format))
At the start: 25 parts, among them P1 ELECTRODES, SW1 PUSH, U1 ADS1299, U2 NRF51822

Commit message: BLE connections
Parts:
- added C17: C, symbol C
- gave numbers to parts that had none: 12
- renumbered BATTERY to BATTERY1, C4 to C10, C3 to C11, C5 to C12, C6 to C14, C2 to C9, U1 to U2, U2 to U4
Connections:
- net VDD is gone; now on net DVDD: C16.1, U3.1 (VOUT)
- net DVDD: now also U4.13 (VSS), U4.35 (AVDD), U4.36 (AVDD); no longer U4.1 (VDD)
- net GND: now also U2.31 (RESV1), U4.23 (SWDIO/RESET), U4.24 (SDWCLK), C17.1; no longer U2.37 (CLK), U2.41 (DAISY_IN), U2.42 (GPIO1), U2.44 (GPIO2), U2.45 (GPIO3), U2.46 (GPIO4), U4.13 (VSS), U4.33 (VSS)
- net at C10.2, C12.2, C14.2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: no longer U2.31 (RESV1)
- net at U2.34 (DIN): now also U4.28 (P0.20); no longer U4.21 (P0.15)
- net at U2.35 (~PWDN~): now also U4.27 (P0.19); no longer U4.20 (P0.14)
- net at U2.36 (~RESET~): now also U4.26 (P0.18); no longer U4.19 (P0.13)
- net at U2.38 (START): now also U4.22 (P0.16); no longer U4.18 (P0.12)
- net at U2.39 (~CS~): now also U4.21 (P0.15); no longer U4.17 (P0.11)
- net at U2.40 (SCLK): now also U4.20 (P0.14); no longer U4.16 (P0.10)
- net at U2.43 (DOUT): now also U4.17 (P0.11); no longer U4.15 (P0.9)
- net at U4.14 (P0.8): now also U2.46 (GPIO4); no longer U2.47 (~DRDY~)
- net at U4.11 (P0.7): now also U2.47 (~DRDY~)
- net at U4.25 (P0.17): now also U2.37 (CLK)
- new net: U2.41 (DAISY_IN), U4.19 (P0.13)
- new net: U2.42 (GPIO1), U4.18 (P0.12)
- new net: U2.44 (GPIO2), U4.16 (P0.10)
- new net: U2.45 (GPIO3), U4.15 (P0.9)
- new net: C17.2, U4.33 (VSS)
- no-connect marks 8 -> 24
Other:
- moved on the sheet: BATTERY1, D1, SW1

Commit message: Schematics updates
Parts:
- C1: value 10nF -> 1nF
Connections:
- net DVDD: now also U2.52 (CLKSEL), U4.1 (VDD)
- net GND: now also U2.41 (DAISY_IN), U2.42 (GPIO1), U2.44 (GPIO2), U2.45 (GPIO3), U2.46 (GPIO4), U4.10 (P0.6/AIN7/AREF1), U4.11 (P0.7), U4.25 (P0.17), U4.26 (P0.18), U4.27 (P0.19), U4.28 (P0.20), U4.3 (P0.30), U4.4 (P0.0/AREF0), U4.5 (P0.1/AIN2), U4.6 (P0.2/AIN3), U4.7 (P0.3/AIN4), U4.8 (P0.4/AIN5), U4.9 (P0.5/AIN6); no longer U2.52 (CLKSEL)
- net at U2.34 (DIN): now also U4.22 (P0.16); no longer U4.28 (P0.20)
- net at U2.35 (~PWDN~): now also U4.21 (P0.15); no longer U4.27 (P0.19)
- net at U2.36 (~RESET~): now also U4.20 (P0.14); no longer U4.26 (P0.18)
- net at U2.37 (CLK): now also U4.19 (P0.13); no longer U4.25 (P0.17)
- net at U2.38 (START): now also U4.18 (P0.12); no longer U4.22 (P0.16)
- net at U2.39 (~CS~): now also U4.17 (P0.11); no longer U4.21 (P0.15)
- net at U2.40 (SCLK): now also U4.16 (P0.10); no longer U4.20 (P0.14)
- net at U2.43 (DOUT): now also U4.15 (P0.9); no longer U4.17 (P0.11)
- net at U4.14 (P0.8): now also U2.47 (~DRDY~); no longer U2.46 (GPIO4)
- net at U2.62 (BIASIN): now also C1.1, R1.1, U2.63 (BIASOUT)
- no-connect marks 24 -> 11
Other:
- note added: "1 - internal\nclock"
- note removed: "Connect to something or \nto leave open?"
- note removed: "Do I need BIASREf?\nAdvantages over internal?"

Commit message: Just ADS1299
Parts:
- removed C17: C, symbol C
- removed U4: NRF51822, symbol NRF51822
Connections:
- net DVDD: now also U2.36 (~RESET~)
- net GND: now also U2.37 (CLK), U2.38 (START)
- net SPI_DIN: now reaches U2.34 (DIN)
- net PWDN: now reaches U2.35 (~PWDN~)
- net SPI_CS: now reaches U2.39 (~CS~)
- net SPI_CLK: now reaches U2.40 (SCLK)
- net SPI_OUT: now reaches U2.43 (DOUT)
- net DRDY: now reaches U2.47 (~DRDY~)
- no-connect marks 11 -> 7
Other:
- note added: "3.3v"
- note added: "5V"
- note removed: "3.3v (regulated)"
- note removed: "5V (regulated)"
- moved on the sheet: BATTERY1, C13, C15, C16, C4, D1, SW1, U1, U3

Commit message: Added note
Other:
- note added: "Interface (decoupled)"
Changed lines of the file:
@@
 Wire Wire Line
 	5650 3100 5300 3100
-Wire Wire Line
-	5300 3500 6300 3500
 Connection ~ 5400 3700
 Connection ~ 4450 1450
@@
 	5300 2300 5500 2300
 Wire Wire Line
-	5500 2300 5500 2400
-Wire Wire Line
-	5500 2400 6300 2400
-Text GLabel 6300 2400 2    60   Input ~ 0
+	5500 2300 5500 2550
+Text GLabel 6300 2550 2    60   Input ~ 0
 DRDY
 Text GLabel 6300 2050 2    60   Input ~ 0
@@
 Text GLabel 6300 3000 2    60   Input ~ 0
 SPI_DIN
-Text GLabel 6300 3500 2    60   Input ~ 0
+Text GLabel 6300 3200 2    60   Input ~ 0
 PWDN
 Wire Wire Line
@@
 Wire Wire Line
 	6300 2050 5400 2050
+Wire Wire Line
+	5500 2550 6300 2550
+Wire Wire Line
+	6300 3200 5950 3200
+Wire Wire Line
+	5950 3200 5950 3500
+Wire Wire Line
+	5950 3500 5300 3500
+Wire Notes Line
+	6200 2400 6200 3400
+Wire Notes Line
+	6200 3400 6850 3400
+Wire Notes Line
+	6850 3400 6850 2400
+Wire Notes Line
+	6850 2400 6200 2400
+Text Notes 6250 3350 0    31   ~ 0
+Interface (decoupled)
 $EndSCHEMATC
